File: Circuito fuente.kicad_pcb (KiCad board)
At the start: 2 copper layers, 99.1 x 99 mm, 37 parts, among them Q1 TIP122, U1 Bornera_1x3, U2 Bornera_1x2, U3 Bornera_1x3, U35 LM7812_TO220, U39 LM7912_TO220, U4 LM7812_TO220, U40 LM7805_TO220, U41 LM7905_TO220, U45 LD1117S12TR_SOT223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

Commit message: Version V1 (Schematic + clearence)
Routing:
- net /-5V: track 47.4 -> 79.1 mm
- net /+12V1: track 60.3 -> 66.5 mm
